File: CAN_Channel.kicad_sch (KiCad schematic)
At the start: 7 parts, among them J1 Conn_01x01, U2 TJA1051T-3

Commit message: complete schematic, initial board layout
Parts:
- renumbered C9 to C13, C10 to C14, C8 to C15, J1 to J3, R1 to R6, S1 to S4
Changed lines of the file:
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@@
 		(dnp no)
 		(fields_autoplaced yes)
-		(property "Reference" "#PWR08"
+		(property "Reference" "#PWR019"
 			(at 62.23 76.2 0)
 			(effects
@@
 			(project "LV3-Core"
 				(path "/f2bb7816-6b2a-47fd-8906-eb4aedd6f9e6/61479cd4-0d84-48d3-a2a5-35c815fbc6c8/26a5cdba-a2c0-4c6f-9b9d-6ff8cc92f2cc"
-					(reference "#PWR08")
-					(unit 1)
-				)
-				(path "/f2bb7816-6b2a-47fd-8906-eb4aedd6f9e6/61479cd4-0d84-48d3-a2a5-35c815fbc6c8/c32bdeb1-5e70-4ff4-b15f-44da73f7e017"
-					(reference "#PWR011")
+					(reference "#PWR019")
+					(unit 1)
+				)
+				(path "/f2bb7816-6b2a-47fd-8906-eb4aedd6f9e6/61479cd4-0d84-48d3-a2a5-35c815fbc6c8/c32bdeb1-5e70-4ff4-b15f-44da73f7e017"
+					(reference "#PWR028")
 					(unit 1)
 				)
@@
 		(dnp no)
 		(fields_autoplaced yes)
-		(property "Reference" "#PWR010"
+		(property "Reference" "#PWR018"
 			(at 139.7 59.69 0)
 			(effects
@@
 			(project "LV3-Core"
 				(path "/f2bb7816-6b2a-47fd-8906-eb4aedd6f9e6/61479cd4-0d84-48d3-a2a5-35c815fbc6c8/26a5cdba-a2c0-4c6f-9b9d-6ff8cc92f2cc"
-					(reference "#PWR010")
-					(unit 1)
-				)
-				(path "/f2bb7816-6b2a-47fd-8906-eb4aedd6f9e6/61479cd4-0d84-48d3-a2a5-35c815fbc6c8/c32bdeb1-5e70-4ff4-b15f-44da73f7e017"
-					(reference "#PWR013")
+					(reference "#PWR018")
+					(unit 1)
+				)
+				(path "/f2bb7816-6b2a-47fd-8906-eb4aedd6f9e6/61479cd4-0d84-48d3-a2a5-35c815fbc6c8/c32bdeb1-5e70-4ff4-b15f-44da73f7e017"
+					(reference "#PWR027")
 					(unit 1)
 				)
@@
 		(dnp no)
 		(fields_autoplaced yes)
-		(property "Reference" "C9"
+		(property "Reference" "C13"
 			(at 130.81 59.6899 0)
 			(effects
@@
 			(project "LV3-Core"
 				(path "/f2bb7816-6b2a-47fd-8906-eb4aedd6f9e6/61479cd4-0d84-48d3-a2a5-35c815fbc6c8/26a5cdba-a2c0-4c6f-9b9d-6ff8cc92f2cc"
-					(reference "C9")
-					(unit 1)
-				)
-				(path "/f2bb7816-6b2a-47fd-8906-eb4aedd6f9e6/61479cd4-0d84-48d3-a2a5-35c815fbc6c8/c32bdeb1-5e70-4ff4-b15f-44da73f7e017"
-					(reference "C12")
+					(reference "C13")
+					(unit 1)
+				)
+				(path "/f2bb7816-6b2a-47fd-8906-eb4aedd6f9e6/61479cd4-0d84-48d3-a2a5-35c815fbc6c8/c32bdeb1-5e70-4ff4-b15f-44da73f7e017"
+					(reference "C16")
 					(unit 1)
 				)
@@
 		(dnp no)
 		(fields_autoplaced yes)
-		(property "Reference" "C10"
+		(property "Reference" "C14"
 			(at 143.51 59.6899 0)
 			(effects
@@
 			(project "LV3-Core"
 				(path "/f2bb7816-6b2a-47fd-8906-eb4aedd6f9e6/61479cd4-0d84-48d3-a2a5-35c815fbc6c8/26a5cdba-a2c0-4c6f-9b9d-6ff8cc92f2cc"
-					(reference "C10")
-					(unit 1)
-				)
-				(path "/f2bb7816-6b2a-47fd-8906-eb4aedd6f9e6/61479cd4-0d84-48d3-a2a5-35c815fbc6c8/c32bdeb1-5e70-4ff4-b15f-44da73f7e017"
-					(reference "C13")
+					(reference "C14")
+					(unit 1)
+				)
+				(path "/f2bb7816-6b2a-47fd-8906-eb4aedd6f9e6/61479cd4-0d84-48d3-a2a5-35c815fbc6c8/c32bdeb1-5e70-4ff4-b15f-44da73f7e017"
+					(reference "C17")
 					(unit 1)
 				)
@@
 		(dnp no)
 		(fields_autoplaced yes)
-		(property "Reference" "J1"
+		(property "Reference" "J3"
 			(at 78.74 71.12 0)
 			(effects
@@
 			(project "LV3-Core"
 				(path "/f2bb7816-6b2a-47fd-8906-eb4aedd6f9e6/61479cd4-0d84-48d3-a2a5-35c815fbc6c8/26a5cdba-a2c0-4c6f-9b9d-6ff8cc92f2cc"
-					(reference "J1")
-					(unit 1)
-				)
-				(path "/f2bb7816-6b2a-47fd-8906-eb4aedd6f9e6/61479cd4-0d84-48d3-a2a5-35c815fbc6c8/c32bdeb1-5e70-4ff4-b15f-44da73f7e017"
-					(reference "J2")
+					(reference "J3")
+					(unit 1)
+				)
+				(path "/f2bb7816-6b2a-47fd-8906-eb4aedd6f9e6/61479cd4-0d84-48d3-a2a5-35c815fbc6c8/c32bdeb1-5e70-4ff4-b15f-44da73f7e017"
+					(reference "J7")
 					(unit 1)
 				)
@@
 		(dnp no)
 		(fields_autoplaced yes)
-		(property "Reference" "#PWR09"
+		(property "Reference" "#PWR020"
 			(at 106.68 90.17 0)
 			(effects
@@
 			(project "LV3-Core"
 				(path "/f2bb7816-6b2a-47fd-8906-eb4aedd6f9e6/61479cd4-0d84-48d3-a2a5-35c815fbc6c8/26a5cdba-a2c0-4c6f-9b9d-6ff8cc92f2cc"
-					(reference "#PWR09")
-					(unit 1)
-				)
-				(path "/f2bb7816-6b2a-47fd-8906-eb4aedd6f9e6/61479cd4-0d84-48d3-a2a5-35c815fbc6c8/c32bdeb1-5e70-4ff4-b15f-44da73f7e017"
-					(reference "#PWR012")
+					(reference "#PWR020")
+					(unit 1)
+				)
+				(path "/f2bb7816-6b2a-47fd-8906-eb4aedd6f9e6/61479cd4-0d84-48d3-a2a5-35c815fbc6c8/c32bdeb1-5e70-4ff4-b15f-44da73f7e017"
+					(reference "#PWR029")
 					(unit 1)
 				)
@@
 		(dnp no)
 		(fields_autoplaced yes)
-		(property "Reference" "R1"
+		(property "Reference" "R6"
 			(at 168.91 67.31 90)
 			(effects
@@
 			(project "LV3-Core"
 				(path "/f2bb7816-6b2a-47fd-8906-eb4aedd6f9e6/61479cd4-0d84-48d3-a2a5-35c815fbc6c8/26a5cdba-a2c0-4c6f-9b9d-6ff8cc92f2cc"
-					(reference "R1")
-					(unit 1)
-				)
-				(path "/f2bb7816-6b2a-47fd-8906-eb4aedd6f9e6/61479cd4-0d84-48d3-a2a5-35c815fbc6c8/c32bdeb1-5e70-4ff4-b15f-44da73f7e017"
-					(reference "R2")
+					(reference "R6")
+					(unit 1)
+				)
+				(path "/f2bb7816-6b2a-47fd-8906-eb4aedd6f9e6/61479cd4-0d84-48d3-a2a5-35c815fbc6c8/c32bdeb1-5e70-4ff4-b15f-44da73f7e017"
+					(reference "R7")
 					(unit 1)
 				)
@@
 		(dnp no)
 		(fields_autoplaced yes)
-		(property "Reference" "C8"
+		(property "Reference" "C15"
 			(at 66.04 77.4699 0)
 			(effects
@@
 			(project "LV3-Core"
 				(path "/f2bb7816-6b2a-47fd-8906-eb4aedd6f9e6/61479cd4-0d84-48d3-a2a5-35c815fbc6c8/26a5cdba-a2c0-4c6f-9b9d-6ff8cc92f2cc"
-					(reference "C8")
-					(unit 1)
-				)
-				(path "/f2bb7816-6b2a-47fd-8906-eb4aedd6f9e6/61479cd4-0d84-48d3-a2a5-35c815fbc6c8/c32bdeb1-5e70-4ff4-b15f-44da73f7e017"
-					(reference "C11")
+					(reference "C15")
+					(unit 1)
+				)
+				(path "/f2bb7816-6b2a-47fd-8906-eb4aedd6f9e6/61479cd4-0d84-48d3-a2a5-35c815fbc6c8/c32bdeb1-5e70-4ff4-b15f-44da73f7e017"
+					(reference "C18")
 					(unit 1)
 				)
@@
 		(dnp no)
 		(fields_autoplaced yes)
-		(property "Reference" "S1"
+		(property "Reference" "S4"
 			(at 199.39 69.8499 0)
 			(effects
@@
 			(project "LV3-Core"
 				(path "/f2bb7816-6b2a-47fd-8906-eb4aedd6f9e6/61479cd4-0d84-48d3-a2a5-35c815fbc6c8/26a5cdba-a2c0-4c6f-9b9d-6ff8cc92f2cc"
-					(reference "S1")
-					(unit 1)
-				)
-				(path "/f2bb7816-6b2a-47fd-8906-eb4aedd6f9e6/61479cd4-0d84-48d3-a2a5-35c815fbc6c8/c32bdeb1-5e70-4ff4-b15f-44da73f7e017"
-					(reference "S2")
-					(unit 1)
-				)
+					(reference "S4")
+					(unit 1)
+				)
+				(path "/f2bb7816-6b2a-47fd-8906-eb4aedd6f9e6/61479cd4-0d84-48d3-a2a5-35c815fbc6c8/c32bdeb1-5e70-4ff4-b15f-44da73f7e017"
+					(reference "S5")
+					(unit 1)
+				)

Commit message: layout almost complete
Connections:
- net CAN+: now also R6.1; no longer S4.2 (COM)
- net CAN-: now also S4.2 (COM); no longer R6.1
Changed lines of the file:
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@@
 	(hierarchical_label "CAN-"
 		(shape bidirectional)
-		(at 162.56 73.66 180)
+		(at 180.34 71.12 180)
 		(effects
 			(font
@@
 		(shape output)
 		(at 91.44 69.85 180)
-		(effects
-			(font
-				(size 1.27 1.27)
-			)
-			(justify right)
-		)
-	)
-	(hierarchical_label "CAN+"
-		(shape bidirectional)
-		(at 180.34 71.12 180)
 		(effects
 			(font
@@
 		)
 	)
+	(hierarchical_label "CAN+"
+		(shape bidirectional)
+		(at 162.56 73.66 180)
+		(effects
+			(font
+				(size 1.27 1.27)
+			)
+			(justify right)
+		)
+	)
