File: Indicator_LED.kicad_sch (KiCad schematic)
At the start: 4 parts

Commit message: complete schematic, initial board layout
Parts:
- renumbered D5 to D7, R7 to R15, R6 to R16, R5 to R17
Changed lines of the file:
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@@
 		(on_board yes)
 		(dnp no)
-		(property "Reference" "R6"
+		(property "Reference" "R16"
 			(at 124.46 96.5199 0)
 			(effects
@@
 			(project "LV3-Core"
 				(path "/f2bb7816-6b2a-47fd-8906-eb4aedd6f9e6/5886a42c-8e6b-486c-adaf-d9c5288f3ea7/175bd41f-64cc-4f98-9a5a-1f637274745b"
-					(reference "R9")
-					(unit 1)
-				)
-				(path "/f2bb7816-6b2a-47fd-8906-eb4aedd6f9e6/5886a42c-8e6b-486c-adaf-d9c5288f3ea7/2153eed5-c388-4600-a8e9-b5718df422db"
-					(reference "R6")
+					(reference "R19")
+					(unit 1)
+				)
+				(path "/f2bb7816-6b2a-47fd-8906-eb4aedd6f9e6/5886a42c-8e6b-486c-adaf-d9c5288f3ea7/2153eed5-c388-4600-a8e9-b5718df422db"
+					(reference "R16")
 					(unit 1)
 				)
@@
 		(dnp no)
 		(fields_autoplaced yes)
-		(property "Reference" "D5"
+		(property "Reference" "D7"
 			(at 106.68 80.01 0)
 			(effects
@@
 			(project "LV3-Core"
 				(path "/f2bb7816-6b2a-47fd-8906-eb4aedd6f9e6/5886a42c-8e6b-486c-adaf-d9c5288f3ea7/175bd41f-64cc-4f98-9a5a-1f637274745b"
-					(reference "D6")
-					(unit 1)
-				)
-				(path "/f2bb7816-6b2a-47fd-8906-eb4aedd6f9e6/5886a42c-8e6b-486c-adaf-d9c5288f3ea7/2153eed5-c388-4600-a8e9-b5718df422db"
-					(reference "D5")
+					(reference "D8")
+					(unit 1)
+				)
+				(path "/f2bb7816-6b2a-47fd-8906-eb4aedd6f9e6/5886a42c-8e6b-486c-adaf-d9c5288f3ea7/2153eed5-c388-4600-a8e9-b5718df422db"
+					(reference "D7")
 					(unit 1)
 				)
@@
 		(on_board yes)
 		(dnp no)
-		(property "Reference" "R5"
+		(property "Reference" "R17"
 			(at 116.84 101.5999 0)
 			(effects
@@
 			(project "LV3-Core"
 				(path "/f2bb7816-6b2a-47fd-8906-eb4aedd6f9e6/5886a42c-8e6b-486c-adaf-d9c5288f3ea7/175bd41f-64cc-4f98-9a5a-1f637274745b"
-					(reference "R8")
-					(unit 1)
-				)
-				(path "/f2bb7816-6b2a-47fd-8906-eb4aedd6f9e6/5886a42c-8e6b-486c-adaf-d9c5288f3ea7/2153eed5-c388-4600-a8e9-b5718df422db"
-					(reference "R5")
+					(reference "R20")
+					(unit 1)
+				)
+				(path "/f2bb7816-6b2a-47fd-8906-eb4aedd6f9e6/5886a42c-8e6b-486c-adaf-d9c5288f3ea7/2153eed5-c388-4600-a8e9-b5718df422db"
+					(reference "R17")
 					(unit 1)
 				)
@@
 		(on_board yes)
 		(dnp no)
-		(property "Reference" "R7"
+		(property "Reference" "R15"
 			(at 132.08 91.4399 0)
 			(effects
@@
 			(project "LV3-Core"
 				(path "/f2bb7816-6b2a-47fd-8906-eb4aedd6f9e6/5886a42c-8e6b-486c-adaf-d9c5288f3ea7/175bd41f-64cc-4f98-9a5a-1f637274745b"
-					(reference "R10")
-					(unit 1)
-				)
-				(path "/f2bb7816-6b2a-47fd-8906-eb4aedd6f9e6/5886a42c-8e6b-486c-adaf-d9c5288f3ea7/2153eed5-c388-4600-a8e9-b5718df422db"
-					(reference "R7")
+					(reference "R18")
+					(unit 1)
+				)
+				(path "/f2bb7816-6b2a-47fd-8906-eb4aedd6f9e6/5886a42c-8e6b-486c-adaf-d9c5288f3ea7/2153eed5-c388-4600-a8e9-b5718df422db"
+					(reference "R15")
 					(unit 1)
 				)
@@
 		(dnp no)
 		(fields_autoplaced yes)
-		(property "Reference" "#PWR"
+		(property "Reference" "#PWR045"
 			(at 114.3 113.03 0)
 			(effects
@@
 			(project "LV3-Core"
 				(path "/f2bb7816-6b2a-47fd-8906-eb4aedd6f9e6/5886a42c-8e6b-486c-adaf-d9c5288f3ea7/175bd41f-64cc-4f98-9a5a-1f637274745b"
-					(reference "#PWR029")
-					(unit 1)
-				)
+					(reference "#PWR046")
+					(unit 1)
+				)
+				(path "/f2bb7816-6b2a-47fd-8906-eb4aedd6f9e6/5886a42c-8e6b-486c-adaf-d9c5288f3ea7/2153eed5-c388-4600-a8e9-b5718df422db"
+					(reference "#PWR045")
+					(unit 1)
+				)

Commit message: minor silkscreen changes, add reverse block diode for 12v ORDER 23 october 2025
Parts:
- R15: value 100 -> 120
Changed lines of the file:
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@@
 			)
 		)
-		(property "Value" "100"
+		(property "Value" "120"
 			(at 132.08 93.9799 0)
 			(effects
